Commit message: Add Ghost

File: sim/rover_description/src/description/pioneer_robot.xacro (robot description, xacro)
@@ -4,7 +4,11 @@
   <xacro:arg name="y_pos" default="0.0"/>
   <xacro:arg name="t_pos" default="0.0"/>
+  <xacro:arg name="r" default="1.0"/>
+  <xacro:arg name="g" default="1.0"/>
+  <xacro:arg name="b" default="1.0"/>
+  <xacro:arg name="a" default="1.0"/>
   <xacro:arg name="mesh_enabled" default="true"/>
   <link name="world"/>
-  <xacro:macro name="p_instance" params="x y theta">
+  <xacro:macro name="p_instance" params="x y theta r g b a">
       <link name="base_link"/>
       <link name="x_axis"/>
@@ -26,4 +30,7 @@
                     scale="0.001 0.001 0.001"/>
             </geometry>
+            <material name="CustomColor">
+              <color rgba="${r} ${g} ${b} ${a}"/>
+            </material>
           </xacro:if>
         </visual>
@@ -47,5 +54,5 @@
         <child link="theta_axis"/>
         <axis xyz="0 0 1"/>
-        <origin xyz="0.0 0.0 0.0" rpy="${theta} ${theta} ${theta}" />
+        <origin xyz="0.0 0.0 0.0" rpy="0.0 0.0 ${theta}" />
         <limit lower="-3" upper="3" effort="0.5" velocity="0.5"/>
       </joint>
@@ -61,4 +68,4 @@
       </joint>
   </xacro:macro>
-  <xacro:p_instance x="$(arg x_pos)" y="$(arg y_pos)" theta="$(arg t_pos)"/>
+  <xacro:p_instance x="$(arg x_pos)" y="$(arg y_pos)" theta="$(arg t_pos)" r="$(arg r)" g="$(arg g)" b="$(arg b)" a="$(arg a)"/>
 </robot>

Commit message: modified: converter
Add set up start-up

Update reference gps

modified: imu

modified: imu

Add Auto setup script for pioneer

Add Auto setup script for pioneer

Add Auto setup script for pioneer

Minor change in convert

Minor change in convert

Add set-up scripts

Bug fix

devide install and setup scripts

File: sim/rover_description/src/description/pioneer_robot.xacro (robot description, xacro)
@@ -41,5 +41,5 @@
         <axis xyz="1 0 0"/>
         <origin xyz="${x} 0.0 0.0" rpy="0 0 0" />
-        <limit lower="-20.0" upper="20.0" effort="0.5" velocity="0.5"/>
+        <limit lower="-200.0" upper="200.0" effort="0.5" velocity="0.5"/>
       </joint>
       <joint name="x_to_y" type="prismatic">
@@ -48,5 +48,5 @@
         <axis xyz="0 1 0"/>
         <origin xyz="0.0 ${y} 0.0" rpy="0 0 0" />
-        <limit lower="-20.0" upper="20.0" effort="0.5" velocity="0.5"/>
+        <limit lower="-200.0" upper="200.0" effort="0.5" velocity="0.5"/>
       </joint>
       <joint name="y_to_t" type="revolute">

Commit message: Reconfigure Sim

File: sim/rover_description/src/description/pioneer_robot.xacro (robot description, xacro)
@@ -1,7 +1,4 @@
 <?xml version="1.0"?>
 <robot xmlns:xacro="http://www.ros.org/wiki/xacro" name="pioneer_rover">
-  <xacro:arg name="x_pos" default="0.0"/>
-  <xacro:arg name="y_pos" default="0.0"/>
-  <xacro:arg name="t_pos" default="0.0"/>
   <xacro:arg name="r" default="1.0"/>
   <xacro:arg name="g" default="1.0"/>
@@ -10,5 +7,5 @@
   <xacro:arg name="mesh_enabled" default="true"/>
   <link name="world"/>
-  <xacro:macro name="p_instance" params="x y theta r g b a">
+  <xacro:macro name="p_instance" params="r g b a">
       <link name="base_link"/>
       <link name="x_axis"/>
@@ -40,5 +37,5 @@
         <child link="x_axis"/>
         <axis xyz="1 0 0"/>
-        <origin xyz="${x} 0.0 0.0" rpy="0 0 0" />
+        <origin xyz="0.0 0.0 0.0" rpy="0 0 0" />
         <limit lower="-200.0" upper="200.0" effort="0.5" velocity="0.5"/>
       </joint>
@@ -47,5 +44,5 @@
         <child link="y_axis"/>
         <axis xyz="0 1 0"/>
-        <origin xyz="0.0 ${y} 0.0" rpy="0 0 0" />
+        <origin xyz="0.0 0.0 0.0" rpy="0 0 0" />
         <limit lower="-200.0" upper="200.0" effort="0.5" velocity="0.5"/>
       </joint>
@@ -54,5 +51,5 @@
         <child link="theta_axis"/>
         <axis xyz="0 0 1"/>
-        <origin xyz="0.0 0.0 0.0" rpy="0.0 0.0 ${theta}" />
+        <origin xyz="0.0 0.0 0.0" rpy="0.0 0.0 0.0" />
         <limit lower="-3" upper="3" effort="0.5" velocity="0.5"/>
       </joint>
@@ -68,4 +65,4 @@
       </joint>
   </xacro:macro>
-  <xacro:p_instance x="$(arg x_pos)" y="$(arg y_pos)" theta="$(arg t_pos)" r="$(arg r)" g="$(arg g)" b="$(arg b)" a="$(arg a)"/>
+  <xacro:p_instance r="$(arg r)" g="$(arg g)" b="$(arg b)" a="$(arg a)"/>
 </robot>

Commit message: Fix Coordinate problem

File: sim/rover_description/src/description/pioneer_robot.xacro (robot description, xacro)
@@ -22,5 +22,5 @@
         <visual>
           <xacro:if value="$(arg mesh_enabled)">
-            <origin xyz="0.0 0.0 0.0" rpy="1.57 0.0 1.57"/>
+            <origin xyz="0.0 0.0 0.0" rpy="1.57 0.0 0.0"/>
             <geometry>
               <mesh filename="package://rover_description/meshes/pioneer_cad_v2.stl"
